File: pcb/eInkFrame.kicad_sch (KiCad schematic)
At the start: 92 parts, among them J1 Socket Raspberry, J2 Socket IT8951, J3 Socket BME680, J40 Socket MPR121 comm, J41 Socket MPR121 contacts, U1 Raspberry, U2 IT8951_Driver, U3 CJMCU-680, U4 MPR121

Commit message: Global doc cleanup, pcb and scripts enhancement, adding images
Parts:
- added HF3: M2.5, MountingHole:MountingHole_2.7mm_M2.5, symbol Mechanical:MountingHole
- HB11, HB21, HM11, HM21: value Nut M2.5 -> Nut M2; footprint MountingHole:MountingHole_2.7mm_M2.5 -> MountingHole:MountingHole_2.7mm_M2; mouser# 144-04M025045HN -> M80-2430000B
- HB12, HB22, HM12, HM22: value Standoff M2.5 -> Standoff M2; footprint MountingHole:MountingHole_2.7mm_M2.5 -> MountingHole:MountingHole_2.7mm_M2; mouser# 761-M2105-2545-AL -> 710-971100244
- HB13, HB23, HM13, HM23: value Screw M2.5 -> Screw M2; footprint MountingHole:MountingHole_2.7mm_M2.5 -> MountingHole:MountingHole_2.7mm_M2; mouser# 534-29300 -> 48SM006
- KT1, KT2, KT3, KT4: footprint eInkFrame:TE 2383945-3 -> eInkFrame:TE 2383945-3 (without clip)
Other:
- moved on the sheet: H1, H11, H12, H13, H2, H21, H22, H23, H3, H31, H32, H33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

Commit message: Change a hard to source component and adapt PCB accordingly + hide some Spotify elements + global formatting
Parts:
- J3: value Socket BME680 -> (none); footprint Connector_PinSocket_2.54mm:PinSocket_1x06_P2.54mm_Vertical_SMD_Pin1Right -> (none)
- KT1, KT2, KT3, KT4: footprint eInkFrame:TE 2383945-3 (without clip) -> eInkFrame:Phoenix contact 1814647; mouser# 571-2383945-3 -> 651-1814647
Changed lines of the file:
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@@
     (property "Reference" "KT1" (id 0) (at 242.57 50.8 0))
     (property "Value" "Screw_Terminal_01x03" (id 1) (at 242.57 53.34 0))
-    (property "Footprint" "eInkFrame:TE 2383945-3 (without clip)" (id 2) (at 229.87 52.07 0)
-      (effects (font (size 1.27 1.27)) hide)
-    )
-    (property "Datasheet" "https://www.mouser.fr/datasheet/2/418/8/ENG_CD_2383945_A1-2451490.pdf" (id 3) (at 229.87 52.07 0)
-      (effects (font (size 1.27 1.27)) hide)
-    )
-    (property "mouser#" "571-2383945-3" (id 4) (at 229.87 52.07 0)
+    (property "Footprint" "eInkFrame:Phoenix contact 1814647" (id 2) (at 229.87 52.07 0)
+      (effects (font (size 1.27 1.27)) hide)
+    )
+    (property "Datasheet" "https://www.mouser.fr/datasheet/2/324/4/1814647-1446675.pdf" (id 3) (at 229.87 52.07 0)
+      (effects (font (size 1.27 1.27)) hide)
+    )
+    (property "mouser#" "651-1814647" (id 4) (at 229.87 52.07 0)
       (effects (font (size 1.27 1.27)) hide)
     )
@@
       (effects (font (size 1.27 1.27)) (justify left))
     )
-    (property "Value" "Socket BME680" (id 1) (at 186.69 99.06 0)
-      (effects (font (size 1.27 1.27)) (justify left))
-    )
-    (property "Footprint" "Connector_PinSocket_2.54mm:PinSocket_1x06_P2.54mm_Vertical_SMD_Pin1Right" (id 2) (at 200.66 121.92 0)
+    (property "Value" "" (id 1) (at 186.69 99.06 0)
+      (effects (font (size 1.27 1.27)) (justify left))
+    )
+    (property "Footprint" "" (id 2) (at 200.66 121.92 0)
       (effects (font (size 1.27 1.27)) hide)
     )
@@
     (property "Reference" "KT4" (id 0) (at 242.57 27.94 0))
     (property "Value" "Screw_Terminal_01x03" (id 1) (at 242.57 30.48 0))
-    (property "Footprint" "eInkFrame:TE 2383945-3 (without clip)" (id 2) (at 229.87 29.21 0)
-      (effects (font (size 1.27 1.27)) hide)
-    )
-    (property "Datasheet" "https://www.mouser.fr/datasheet/2/418/8/ENG_CD_2383945_A1-2451490.pdf" (id 3) (at 229.87 29.21 0)
-      (effects (font (size 1.27 1.27)) hide)
-    )
-    (property "mouser#" "571-2383945-3" (id 4) (at 229.87 29.21 0)
+    (property "Footprint" "eInkFrame:Phoenix contact 1814647" (id 2) (at 229.87 29.21 0)
+      (effects (font (size 1.27 1.27)) hide)
+    )
+    (property "Datasheet" "https://www.mouser.fr/datasheet/2/324/4/1814647-1446675.pdf" (id 3) (at 229.87 29.21 0)
+      (effects (font (size 1.27 1.27)) hide)
+    )
+    (property "mouser#" "651-1814647" (id 4) (at 229.87 29.21 0)
       (effects (font (size 1.27 1.27)) hide)
     )
@@
     (property "Reference" "KT2" (id 0) (at 242.57 43.18 0))
     (property "Value" "Screw_Terminal_01x03" (id 1) (at 242.57 45.72 0))
-    (property "Footprint" "eInkFrame:TE 2383945-3 (without clip)" (id 2) (at 229.87 44.45 0)
-      (effects (font (size 1.27 1.27)) hide)
-    )
-    (property "Datasheet" "https://www.mouser.fr/datasheet/2/418/8/ENG_CD_2383945_A1-2451490.pdf" (id 3) (at 229.87 44.45 0)
-      (effects (font (size 1.27 1.27)) hide)
-    )
-    (property "mouser#" "571-2383945-3" (id 4) (at 229.87 44.45 0)
+    (property "Footprint" "eInkFrame:Phoenix contact 1814647" (id 2) (at 229.87 44.45 0)
+      (effects (font (size 1.27 1.27)) hide)
+    )
+    (property "Datasheet" "https://www.mouser.fr/datasheet/2/324/4/1814647-1446675.pdf" (id 3) (at 229.87 44.45 0)
+      (effects (font (size 1.27 1.27)) hide)
+    )
+    (property "mouser#" "651-1814647" (id 4) (at 229.87 44.45 0)
       (effects (font (size 1.27 1.27)) hide)
     )
@@
     (property "Reference" "KT3" (id 0) (at 242.57 35.56 0))
     (property "Value" "Screw_Terminal_01x03" (id 1) (at 242.57 38.1 0))
-    (property "Footprint" "eInkFrame:TE 2383945-3 (without clip)" (id 2) (at 229.87 36.83 0)
-      (effects (font (size 1.27 1.27)) hide)
-    )
-    (property "Datasheet" "https://www.mouser.fr/datasheet/2/418/8/ENG_CD_2383945_A1-2451490.pdf" (id 3) (at 229.87 36.83 0)
-      (effects (font (size 1.27 1.27)) hide)
-    )
-    (property "mouser#" "571-2383945-3" (id 4) (at 229.87 36.83 0)
+    (property "Footprint" "eInkFrame:Phoenix contact 1814647" (id 2) (at 229.87 36.83 0)
+      (effects (font (size 1.27 1.27)) hide)
+    )
+    (property "Datasheet" "https://www.mouser.fr/datasheet/2/324/4/1814647-1446675.pdf" (id 3) (at 229.87 36.83 0)
+      (effects (font (size 1.27 1.27)) hide)
+    )
+    (property "mouser#" "651-1814647" (id 4) (at 229.87 36.83 0)
       (effects (font (size 1.27 1.27)) hide)
     )
@@
     )
     (path "/5c54fdce-28e8-4f72-bb25-0bf3b6f09690"
-      (reference "J3") (unit 1) (value "Socket BME680") (footprint "Connector_PinSocket_2.54mm:PinSocket_1x06_P2.54mm_Vertical_SMD_Pin1Right")
+      (reference "J3") (unit 1) (value "Socket BME680") (footprint "Connector_PinSocket_2.54mm:PinSocket_1x06_P2.54mm_Vertical_SMD_Pin1Left")
     )
     (path "/6ad55953-7a86-4bfb-a23b-dcf3a404bbd3"
@@
     )
     (path "/0e117404-8b24-4d21-b2a5-695edaee805c"
-      (reference "KT1") (unit 1) (value "Screw_Terminal_01x03") (footprint "eInkFrame:TE 2383945-3 (without clip)")
+      (reference "KT1") (unit 1) (value "Screw_Terminal_01x03") (footprint "eInkFrame:Phoenix contact 1814647")
     )
     (path "/c1eba4b2-7576-4888-9ba8-24fc9a7ff28f"
-      (reference "KT2") (unit 1) (value "Screw_Terminal_01x03") (footprint "eInkFrame:TE 2383945-3 (without clip)")
+      (reference "KT2") (unit 1) (value "Screw_Terminal_01x03") (footprint "eInkFrame:Phoenix contact 1814647")
     )
     (path "/ddce5d33-f931-4b78-8608-df870869e452"
-      (reference "KT3") (unit 1) (value "Screw_Terminal_01x03") (footprint "eInkFrame:TE 2383945-3 (without clip)")
+      (reference "KT3") (unit 1) (value "Screw_Terminal_01x03") (footprint "eInkFrame:Phoenix contact 1814647")
     )
     (path "/a6984c3f-be8e-4c45-b30f-ef2764ac40f9"
-      (reference "KT4") (unit 1) (value "Screw_Terminal_01x03") (footprint "eInkFrame:TE 2383945-3 (without clip)")
+      (reference "KT4") (unit 1) (value "Screw_Terminal_01x03") (footprint "eInkFrame:Phoenix contact 1814647")
     )
     (path "/3528ffbf-299d-477c-a201-66ca2c451755"

Commit message: New PCB stand, adding photos, minor updates after final mounting
Parts:
- removed HF2: M2.5, MountingHole:MountingHole_2.7mm_M2.5, symbol Mechanical:MountingHole
- added HF3, HF4: M3, MountingHole:MountingHole_3.2mm_M3, symbol Mechanical:MountingHole
- HF1: value M2.5 -> M3; footprint MountingHole:MountingHole_2.7mm_M2.5 -> MountingHole:MountingHole_3.2mm_M3
- HF11, HF21: value Nut M2.5 -> Nut M3; footprint MountingHole:MountingHole_2.7mm_M2.5 -> MountingHole:MountingHole_3.2mm_M3; mouser# 144-04M025045HN -> 144-04M030050HN
- HF12, HF22: value Screw M2.5 -> (none); footprint MountingHole:MountingHole_2.7mm_M2.5 -> (none); mouser# 534-29300 -> 5164-SH1000-F
- HF2: renamed from HF3; value M2.5 -> M3; footprint MountingHole:MountingHole_2.7mm_M2.5 -> MountingHole:MountingHole_3.2mm_M3
- J3: value (none) -> Socket BME680; footprint (none) -> Connector_PinSocket_2.54mm:PinSocket_1x06_P2.54mm_Vertical_SMD_Pin1Left
- KT1, KT2, KT3, KT4: value Screw_Terminal_01x03 -> Terminal_01x03; symbol Connector:Screw_Terminal_01x03 -> eInkFrame:Phoenix_contact_1814647
- renumbered HK01 to HK1, HK02 to HK2, HK03 to HK3, HK04 to HK4, HK05 to HK5, HK06 to HK6, HK07 to HK7, HK08 to HK8, HK09 to HK9
Connections:
- net GND: now also KT1.SH1 (SH)
- net at J41.4 (Pin_4), KT1.3 (Pin_3): now also KT2.SH1 (SH)
- net at J41.10 (Pin_10), KT3.3 (Pin_3): now also KT4.SH1 (SH)
- net at J41.11 (Pin_11), KT4.1 (Pin_1): now also KT3.SH2 (SH)
- net at J41.5 (Pin_5), KT2.1 (Pin_1): now also KT1.SH2 (SH)
- net at J41.7 (Pin_7), KT2.3 (Pin_3): now also KT3.SH1 (SH)
- net at J41.8 (Pin_8), KT3.1 (Pin_1): now also KT2.SH2 (SH)
Other:
- note added: "Standoffs height to select according to frame border and inner standoffs To source from: https://mou.sr/3qZdDCO"
- moved on the sheet: E1, E2, H1, H11, H12, H13, H2, H21, H22, H23, H3, H31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
